Commit message: change sensor origin

File: src/erp42_description/urdf/erp42_gazebo.xacro (robot description, xacro)
@@ -116,3 +116,16 @@
     </joint>
   </ros2_control>
+  <gazebo>
+  <plugin name="p3d_base_controller" filename="libgazebo_ros_p3d.so">
+    <ros>
+      <remapping>odom:=odometry/absolute</remapping>
+    </ros>
+    <body_name>base_link</body_name>
+    <frame_name>map</frame_name>
+    <update_rate>30.0</update_rate>
+    <xyz_offset>0 0 0</xyz_offset>
+    <rpy_offset>0 0 0</rpy_offset>
+    <gaussian_noise>0.00</gaussian_noise>
+  </plugin>
+</gazebo>
 </robot>

File: src/erp42_description/urdf/erp42_sensors.xacro (robot description, xacro)
@@ -24,5 +24,5 @@
     <parent link="structure"/>
     <child link="imu_link"/>
-    <origin xyz="0.0 0.0 0.15" rpy="0 0 0"/>
+    <origin xyz="0.0 0.0 1.18" rpy="0 0 0"/>
   </joint>
   <link name="gps_link">
@@ -49,5 +49,5 @@
     <parent link="structure"/>
     <child link="gps_link"/>
-    <origin xyz="0.2 0.0 0.2" rpy="0 0 0"/>
+    <origin xyz="0.0 0.0 1.38" rpy="0 0 0"/>
   </joint>
 </robot>
